File: hardware/BREAD_Slice.kicad_sch (KiCad schematic)
At the start: 15 parts, among them J1 Conn_01x10_Female, U1 AP63205

Commit message: initial commit, schematic and board done
Connections:
- net ORP_IN: now reaches A1.19 (A0)
- no-connect marks 22 -> 21
Other:
- added sheet ORP Amplifier (orp_amp.kicad_sch)
